File: TDR.kicad_pcb (KiCad board)
At the start: 4 copper layers, 80 x 80 mm, 46 parts, among them J1 Conn_Coaxial, J2 Conn_Coaxial, J3 Conn_Coaxial, J4 Conn_Coaxial, J5 Screw_Terminal_01x02, U1 CDCLVC1112PW‎

Commit message: pretty
Parts:
- added FID1: Fiducial, Fiducial:Fiducial_1mm_Mask3mm, F.Cu at (80.0, 54.0)
- added FID2: Fiducial, Fiducial:Fiducial_1mm_Mask3mm, B.Cu at (65.0, 119.0)
- added FID3: Fiducial, Fiducial:Fiducial_1mm_Mask3mm, B.Cu at (120.0, 54.0)
- added FID4: Fiducial, Fiducial:Fiducial_1mm_Mask3mm, F.Cu at (65.0, 119.0)
- added FID5: Fiducial, Fiducial:Fiducial_1mm_Mask3mm, B.Cu at (135.0, 119.0)
- added FID6: Fiducial, Fiducial:Fiducial_1mm_Mask3mm, F.Cu at (120.0, 54.0)
- added FID7: Fiducial, Fiducial:Fiducial_1mm_Mask3mm, F.Cu at (135.0, 119.0)
- added FID8: Fiducial, Fiducial:Fiducial_1mm_Mask3mm, B.Cu at (80.0, 54.0)
- added H1: MountingHole, MountingHole:MountingHole_3.2mm_M3_Pad_Via, F.Cu at (135.0, 125.0)
- added H2: MountingHole, MountingHole:MountingHole_3.2mm_M3_Pad_Via, F.Cu at (74.0, 54.0)
- added H3: MountingHole, MountingHole:MountingHole_3.2mm_M3_Pad_Via, F.Cu at (126.0, 54.0)
- added H4: MountingHole, MountingHole:MountingHole_3.2mm_M3_Pad_Via, F.Cu at (65.0, 125.0)
Other:
- board text added: "TDR 6dB splitter LVCMOS Philippe Trottier © 2022 εr=XX H=XXmm"
