File: TDR.kicad_sch (KiCad schematic)
At the start: 46 parts, among them J1 Conn_Coaxial, J2 Conn_Coaxial, J3 Conn_Coaxial, J4 Conn_Coaxial, U1 CDCLVC1112PW‎

Commit message: pretty
Parts:
- added FID? (x8): Fiducial, Fiducial:Fiducial_1mm_Mask3mm, symbol Mechanical:Fiducial
- added H? (x4): MountingHole, MountingHole:MountingHole_3.2mm_M3_Pad_Via, symbol Mechanical:MountingHole
